File: STM_PCB/STM_PCB.sch (KiCad schematic (older format))
At the start: 26 parts, among them IC1 XC6201P332MR-G, J1 ST_LINK, J2 USB_B_Mini, J3 Conn_01x15, J4 Conn_01x15, J5 DODATKOWE, SW1 SW_Push, SW2 SW_Push, U1 STM32F042K6Tx

Commit message: Signed-off-by: unknown <tomasz@fortec.pl>
Parts:
- removed IC1: XC6201P332MR-G, SOT95P280X130-5N, symbol SamacSys_Parts:XC6201P332MR-G
- removed J2: USB_B_Mini, Connector_USB:USB_Mini-B_Wuerth_65100516121_Horizontal, symbol Connector:USB_B_Mini
- removed RV1: R_POT, Potentiometer_SMD:Potentiometer_ACP_CA6-VSMD_Vertical, symbol Device:R_POT
- added J2: USB_B_Micro, Connector_USB:USB_Micro-B_Molex_47346-0001, symbol Connector:USB_B_Micro
- added U2: LD39015M33R, Package_TO_SOT_SMD:SOT-23-5, symbol Regulator_Linear:LD39015M33R
- J1: footprint (none) -> Connector_PinHeader_2.54mm:PinHeader_1x04_P2.54mm_Vertical
- J3, J4: footprint (none) -> Connector_PinHeader_2.54mm:PinHeader_1x15_P2.54mm_Vertical
- J5: footprint (none) -> Connector_PinHeader_2.54mm:PinHeader_1x02_P2.54mm_Vertical
- R1, R2, R3, R4, R5, R6, R7: footprint Resistor_SMD:R_0612_1632Metric_Pad1.18x3.40mm_HandSolder -> Resistor_SMD:R_0603_1608Metric_Pad0.98x0.95mm_HandSolder
- SW1, SW2: footprint Button_Switch_SMD:SW_Push_1P1T_NO_6x6mm_H9.5mm -> Button_Switch_SMD:SW_Push_1P1T_NO_Vertical_Wuerth_434133025816
Connections:
- net +5V: now also U2.1 (IN), U2.3 (EN)
- net GND: now also J2.5 (GND), J2.6 (Shield), U2.2 (GND)
- net VCC: now also U2.5 (OUT)
- net at FB1.2: now also J2.1 (VBUS)
- net at C2.1, R2.2: now also J2.2 (D-)
- net at C1.1, R1.2: now also J2.3 (D+)
- no-connect marks 3 -> 1
Other:
- moved on the sheet: C4, POWER1, R6
